File: smart_soldering_iron.kicad_sch (KiCad schematic)
At the start: 33 parts, among them U1 ATMEGA328PB-AU

Commit message: code addition
Other:
- added sheet bms_with charging (bms_with_charging.kicad_sch)
- note added: "ssd1306_128*32 display connector only.avoided the bare display for simplicity"
- note removed: "ssd1306_128*32 display"
Changed lines of the file:
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@@
 		)
 	)
-	(text "ssd1306_128*32 display\n"
+	(text "ssd1306_128*32 display connector only.avoided the bare display for simplicity\n"
 		(exclude_from_sim no)
-		(at 207.264 59.436 0)
+		(at 235.204 58.674 0)
 		(effects
 			(font
@@
 				)
 			)
+		)
+	)
+	(sheet
+		(at 39.37 212.09)
+		(size 15.494 3.81)
+		(exclude_from_sim no)
+		(in_bom yes)
+		(on_board yes)
+		(dnp no)
+		(fields_autoplaced yes)
+		(stroke
+			(width 0.1524)
+			(type solid)
+		)
+		(fill
+			(color 0 0 0 0.0000)
+		)
+		(property "Sheetname" "bms_with charging"
+			(at 39.37 211.3784 0)
+			(effects
+				(font
+					(size 1.27 1.27)
+				)
+				(justify left bottom)
+			)
+		)
+		(property "Sheetfile" "bms_with_charging.kicad_sch"
+			(at 39.37 216.4846 0)
+			(effects
+				(font
+					(size 1.27 1.27)
+				)
+				(justify left top)
+			)
+		)
+		(instances
+			(project "smart_soldering_iron"
+				(path "/2df86fbf-058b-45fc-8204-866599907949"
+					(page "3")
+				)
+			)

Commit message: COMPLETED CIRCUIT DIAGRAM
Parts:
- removed R? (x3): 5k, symbol Device:R
- removed U1: ATMEGA328PB-AU, ATMEGA328PB-AU:QFP80P900X900X120-32N, symbol smart_soldering_iron:ATMEGA328PB-AU
- added C26, C31, C32: 100n, Capacitor_SMD:C_0603_1608Metric, symbol Device:C
- added C33: 10u, Capacitor_SMD:C_0603_1608Metric, symbol Device:C
- added R10, R11, R12, R46, R47, R48, R49: 10K, Resistor_SMD:R_0603_1608Metric, symbol Device:R
- added R54: 1K, Resistor_SMD:R_0603_1608Metric, symbol Device:R
- added U8: ~, smart_soldering_iron:ST LIS3DHTR_ACCELEROMETER_LGA-16_L3.0-W3.0-P0.50-TL, symbol smart_soldering_iron:LIS3DHTR_C15134
- C1, C10, C11, C2, C3, C4, C5, C6, C7, C8, C9: renamed from C?; footprint (none) -> Capacitor_SMD:C_0603_1608Metric
- R1, R5, R8, R9: renamed from R?; value 10k -> 10K; footprint (none) -> Resistor_SMD:R_0603_1608Metric
- R2: renamed from R?; value 1.5k -> 1K; footprint (none) -> Resistor_SMD:R_0603_1608Metric
- R3, R7: renamed from R?; value 1k -> 1K; footprint (none) -> Resistor_SMD:R_0603_1608Metric
- R4: renamed from R?; value 200k -> 200K; footprint (none) -> Resistor_SMD:R_0603_1608Metric
- R6: renamed from R?; value 6.2k -> 3.3K; footprint (none) -> Resistor_SMD:R_0603_1608Metric
- U2: renamed from U?; footprint ProLib_pcs_2025-10-03:SOT-23-5_L3.0-W1.7-P0.95-LS2.8-BR -> smart_soldering_iron:LM321_SOT-23-5_L3.0-W1.7-P0.95-LS2.8-BR
- U3: renamed from U?; footprint ATMEGA328P-AU:QFP80P900X900X120-32N -> smart_soldering_iron:ATMEGA328P-AU_QFP80P900X900X120-32N
- Y1: renamed from Y?; value 8 MHZ -> 16 MHZ
- gave numbers to parts that had none: 6
Connections:
- net <_BUTTON: now also C10.2, SW2.1, U3.2 (PD4), R11.1; no longer U3.13 (PB1)
- net >_BUTTON: now also C11.2, SW3.1, U3.1 (PD3), R12.1; no longer U3.12 (PB0)
- net GND: now also C26.1, C31.2, C32.1, C33.1, R49.1, U8.10 (RES), U8.12 (GND), U8.5 (GND)
- net OK_BUTTON: now also C9.2, SW1.1, U3.14 (PB2), R10.1; no longer U3.2 (PD4)
- net SCL: now also R46.1, U8.4 (SCL/SPC)
- net SDA: now also R47.1, U8.6 (SDA/SDI/SDO)
- net TIP_MOS: now reaches U3.15 (PB3)
- net BALANCE_HIGH_MOS: now reaches U3.16 (PB4)
- net BALANCE_LOW_MOS: now reaches U3.17 (PB5)
- net B1_SENSE: now reaches U3.25 (PC2)
- net B2_SENSE: now reaches U3.26 (PC3)
- net LIS3DHTR_INT: now reaches U3.32 (PD2)
- net LIS3DHTR_INT: now also R54.1
- net D0_rxd renamed D0_RXD
- net D1_txd renamed D1_TXD
- net P+ renamed TIP+
- net cfg1 renamed CFG1
- net cfg2 renamed CFG2
- net cfg3 renamed CFG3
- net temp_sense renamed TEMP_SENSE
- net v_sense renamed V_SENSE
- net V_SENSE: now also C31.1
- net vcc_5v renamed VCC_5V
- net VCC_5V: now also R10.2, R11.2, R12.2
- new net: R48.1, R49.2, U8.7 (SDO/SA0)
- new net: R54.2, U8.11 (INT1)
- new net CHARG_STAT: U3.13 (PB1)
- new net LATCH_OFF_MCU: U3.12 (PB0)
- new net TIP_AMP_SENSE: U8.16 (ADC1)
- new net VCC_3V3: C26.2, C32.2, C33.2, R46.2, R47.2, R48.2, U8.1 (VDD_IO), U8.14 (VDD), U8.8 (CS)
- no-connect marks 9 -> 16
Other:
- sheet bms_with charging renamed battery
- sheet sheet_2 renamed power
- sheet battery: file bms_with_charging.kicad_sch -> bms_with_charging.Kicad_sch
- sheet power: file sheet_2.kicad_sch -> sheet_2.Kicad_sch
- note added: "make sure the pullup on the arduino i2c is disabled before soldering LIS3DHTR"
- moved on the sheet: C1, C10, C11, C3, C4, C5, C6, C8, C9, D2, J1, R2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
