File: bms_with_charging.kicad_sch (KiCad schematic)
At the start: 8 parts

Commit message: code addition
Parts:
- added Q?: ~, ProLib_pcs_2025-10-03:DFN-8_L3.0-W3.0-P0.65-BL, symbol smart_soldering_iron:AON7410
- added R?: 100k, symbol Device:R
- added R? (x2): 1k, symbol Device:R
- added R?: R, symbol Device:R
Connections:
- net GND: now also Q?.1 (S), Q?.2 (S), Q?.3 (S), R?.2
- net at Q?.4 (G): now also R?.2
- net at Q?.5 (D): now also Q?.6 (D), Q?.7 (D), Q?.8 (D), Q?.9 (D)
- new net: Q?.4 (G), R?.1
- new net: Q?.1 (S), Q?.2 (S), Q?.3 (S), R?.1
- new net m_g_char: R?.2, R?.2
- new net m_g_disch: R?.1, R?.1
Other:
- moved on the sheet: Q?

Commit message: COMPLETED CIRCUIT DIAGRAM
Parts:
- removed J?: Conn_01x04_Pin, symbol Connector:Conn_01x04_Pin
- removed Q? (x2): ~, ProLib_pcs_2025-10-03:DFN-8_L3.0-W3.0-P0.65-BL, symbol smart_soldering_iron:AON7410
- removed R? (x7): R, symbol Device:R
- removed R?: 100k, symbol Device:R
- removed R? (x2): 1k, symbol Device:R
- added C23, C24: 10u, Capacitor_SMD:C_0603_1608Metric, symbol Device:C
- added C29, C30: 100n, Capacitor_SMD:C_0603_1608Metric, symbol Device:C
- added D10, D9: D_Zener, symbol Device:D_Zener
- added D4, D5: LED, symbol Device:LED
- added D6, D8: D_SchottKy, symbol Device:D_Schottky
- added J2: Conn_01x03_SocKet, symbol Connector:Conn_01x03_Socket
- added L2: 4.7u, symbol Device:L
- added Q1, Q4: ~, smart_soldering_iron:S8050_TRANSIS_25V_0.5A_npn_SOT-23-3_L2.9-W1.3-P1.90-LS2.4-BR, symbol smart_soldering_iron:S8050
- added Q2, Q9: ~, smart_soldering_iron:LGE AO3401_P_MOS_SOT-23-3_L2.9-W1.6-P1.90-LS2.8-BR, symbol smart_soldering_iron:AO3401_C688915
- added Q3: ~, smart_soldering_iron:d03400d_N_MOS_SOT-23-3_L2.9-W1.6-P1.90-LS2.8-BR, symbol smart_soldering_iron:DO3400D
- added Q5, Q7: ~, ProLib_pcs_2025-11-05:SOT-23-3_L2.9-W1.3-P1.90-LS2.4-BR, symbol smart_soldering_iron:PMBT2907A,215
- added Q6: ~, ProLib_pcs_2025-11-06:PDFN-8_L3.1-W3.0-P0.65-LS3.3-BL, symbol smart_soldering_iron:DOZ30P03
- added Q8: ~, ProLib_pcs_2025-10-03:DFN-8_L3.0-W3.0-P0.65-BL, symbol smart_soldering_iron:AON7410
- added R20, R21, R23, R24, R25, R28, R31, R33, R38, R39, R41, R42: 10K, Resistor_SMD:R_0603_1608Metric, symbol Device:R
- added R22, R26, R45: 100K, Resistor_SMD:R_0603_1608Metric, symbol Device:R
- added R27: 50, symbol Device:R
- added R29, R30, R32, R34, R40: 2.2K, Resistor_SMD:R_0603_1608Metric, symbol Device:R
- added R35, R36: 1K, Resistor_SMD:R_0603_1608Metric, symbol Device:R
- added R37: 0.06, symbol Device:R
- added U1: ~, smart_soldering_iron:CN3302_SOP-8_L4.9-W3.9-P1.27-LS6.0-BL, symbol smart_soldering_iron:CN3302
Connections:
- net GND: now also C23.2, C24.2, C29.2, C30.2, D5.1 (K), D9.2 (A), J2.3 (Pin_3), Q1.2 (E), Q3.2 (S), Q4.2 (E), Q8.1 (S), Q8.2 (S), Q8.3 (S), R21.2, R26.1, R32.1, U1.4 (GND)
- new net: R20.2, R21.1, R45.2
- new net: Q4.1 (B), R42.2
- new net: Q4.3 (C), R29.1, R30.1, R40.2
- new net: D6.2 (A), L2.2, Q8.5 (D), Q8.6 (D), Q8.7 (D), Q8.8 (D), Q8.9 (D)
- new net: Q5.1 (B), R30.2
- new net: Q5.3 (C), R31.2, R32.2, R34.2
- new net: D10.2 (A), R28.2
- new net: C23.1, D8.2 (A), Q6.5 (D), Q6.6 (D), Q6.7 (D), Q6.8 (D), Q6.9 (D), R36.2, R37.1, U1.2 (CE), U1.7 (VIN)
- new net: Q6.4 (G), R34.1
- new net: Q3.1 (G), R23.2
- new net: Q2.3 (D), Q3.3 (D), R27.1
- new net: D4.2 (A), R36.1
- new net: Q1.3 (C), R24.1, R25.1
- new net: L2.1, R37.2, U1.8 (CSN)
- new net: Q2.1 (G), R25.2
- new net: Q1.1 (B), R38.2
- new net: Q7.1 (B), R41.2
- new net: Q7.3 (C), R33.2
- new net: D4.1 (K), R35.2, R39.2, U1.1 (STAT)
- new net: Q8.4 (G), U1.5 (LDRV)
- new net: Q9.1 (G), R40.1
- new net: D5.2 (A), R35.1
- new net 1S: J2.2 (Pin_2), Q7.2 (E), R22.2, R27.2
- new net 2S: C24.1, D6.1 (K), J2.1 (Pin_1), Q2.2 (S), Q5.2 (E), Q9.2 (S), R20.1, R24.2, R29.2, U1.3 (BAT)
- new net 2S_MOS_OUT: Q9.3 (D)
- new net B1_SENSE: C29.1, R22.1
- new net B2_SENSE: C30.1, R45.1
- new net BALANCE_HIGH_MOS: R38.1
- new net BALANCE_LOW_MOS: R23.1, R26.2
- new net CHARG_STAT: R39.1
- new net LATCH_OFF_MCU: D9.1 (K), R28.1, R31.1, R33.1, R42.1
- new net OK_BUTTON: R41.1
- new net VCC_5V: D8.1 (K)
- new net Vin: D10.1 (K), Q6.1 (S), Q6.2 (S), Q6.3 (S)
- no-connect marks 0 -> 1
Other:
- note added: ">pressing OK_BUTTON latches the mosfet in on state until the mcu turns it off. This is also useful when the battery voltage is low >5v zener turn on the bjt and turn of the charger mosfet"
- note added: "NOTES 1.GND is battery ground 2.GND is higher potential after the mosfet drop 3.B1_SENSE not using divider becausethe voltage is below 5v"
- note added: "This circuit balances the voltage across the 2 battery by dissipating power in the 50ohm resistor 50ohm is an random logical value"
