File: sheet_2.kicad_sch (KiCad schematic)
At the start: 24 parts

Commit message: code addition
Parts:
- added R?: 1k, symbol Device:R
Connections:
- net RESET: now also R?.1
- net vcc_5v: now also R?.2
Changed lines of the file:
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@@
 		(exclude_from_sim no)
 		(at 33.02 91.44 0)
-		(size 90.932 45.974)
+		(size 93.472 45.974)
 		(margins 0.9525 0.9525 0.9525 0.9525)
 		(stroke
@@
 	)
 	(junction
+		(at 105.41 114.3)
+		(diameter 0)
+		(color 0 0 0 0)
+	)
+	(junction
 		(at 54.61 106.68)
 		(diameter 0)
@@
 	(wire
 		(pts
+			(xy 105.41 121.92) (xy 105.41 123.19)
+		)
+		(stroke
+			(width 0)
+			(type default)
+		)
+	)
+	(wire
+		(pts
 			(xy 52.07 105.41) (xy 52.07 106.68)
 		)
@@
 	(wire
 		(pts
-			(xy 101.6 114.3) (xy 104.14 114.3)
+			(xy 101.6 114.3) (xy 105.41 114.3)
 		)
 		(stroke
@@
 	(wire
 		(pts
+			(xy 105.41 123.19) (xy 121.92 123.19)
+		)
+		(stroke
+			(width 0)
+			(type default)
+		)
+	)
+	(wire
+		(pts
 			(xy 270.51 73.66) (xy 270.51 77.47)
 		)
@@
 	(wire
 		(pts
+			(xy 121.92 123.19) (xy 121.92 118.11)
+		)
+		(stroke
+			(width 0)
+			(type default)
+		)
+	)
+	(wire
+		(pts
+			(xy 105.41 114.3) (xy 109.22 114.3)
+		)
+		(stroke
+			(width 0)
+			(type default)
+		)
+	)
+	(wire
+		(pts
 			(xy 101.6 109.22) (xy 106.68 109.22)
 		)
@@
 	(global_label "RESET"
 		(shape input)
-		(at 104.14 114.3 0)
+		(at 109.22 114.3 0)
 		(fields_autoplaced yes)
 		(effects
@@
 		)
 		(property "Intersheetrefs" "${INTERSHEET_REFS}"
-			(at 112.8703 114.3 0)
+			(at 117.9503 114.3 0)
 			(effects
 				(font
@@
 	)
 	(symbol
+		(lib_id "power:VCC")
+		(at 121.92 118.11 0)
+		(unit 1)
+		(exclude_from_sim no)
+		(in_bom yes)
+		(on_board yes)
+		(dnp no)
+		(fields_autoplaced yes)
+		(property "Reference" "#PWR058"
+			(at 121.92 121.92 0)
+			(effects
+				(font
+					(size 1.27 1.27)
+				)
+				(hide yes)
+			)
+		)
+		(property "Value" "vcc_5v"
+			(at 121.92 113.03 0)
+			(effects
+				(font
+					(size 1.27 1.27)
+				)
+			)
+		)
+		(property "Footprint" ""
+			(at 121.92 118.11 0)
+			(effects
+				(font
+					(size 1.27 1.27)
+				)
+				(hide yes)
+			)
+		)
+		(property "Datasheet" ""
+			(at 121.92 118.11 0)
+			(effects
+				(font
+					(size 1.27 1.27)
+				)
+				(hide yes)
+			)
+		)
+		(property "Description" "Power symbol creates a global label with name \"VCC\""
+			(at 121.92 118.11 0)
+			(effects
+				(font
+					(size 1.27 1.27)
+				)
+				(hide yes)
+			)
+		)
+		(pin "1"
+		)
+		(instances
+			(project "smart_soldering_iron"
+				(path "/2df86fbf-058b-45fc-8204-866599907949/63b7c06e-9066-41e6-8478-c4bea396f7f1"
+					(reference "#PWR058")
+					(unit 1)
+				)
+			)
+		)
+	)
+	(symbol
 		(lib_id "Device:C")
 		(at 196.85 36.83 0)
@@
 					(unit 1)
 				)
+			)
+		)
+	)
+	(symbol
+		(lib_id "Device:R")
+		(at 105.41 118.11 0)
+		(unit 1)
+		(exclude_from_sim no)
+		(in_bom yes)
+		(on_board yes)
+		(dnp no)
+		(property "Reference" "R?"
+			(at 108.712 116.332 0)
+			(effects
+				(font
+					(size 1.27 1.27)
+				)
+			)
+		)
+		(property "Value" "1k"
+			(at 108.712 118.872 0)
+			(effects
+				(font
+					(size 1.27 1.27)
+				)
+			)
+		)
+		(property "Footprint" ""
+			(at 103.632 118.11 90)
+			(effects
+				(font
+					(size 1.27 1.27)
+				)
+				(hide yes)
+			)
+		)
+		(property "Datasheet" "~"
+			(at 105.41 118.11 0)
+			(effects
+				(font
+					(size 1.27 1.27)
+				)
+				(hide yes)
+			)
+		)
+		(property "Description" "Resistor"
+			(at 105.41 118.11 0)
+			(effects
+				(font
+					(size 1.27 1.27)
+				)
+				(hide yes)
+			)
+		)
+		(pin "1"
+		)
+		(pin "2"
+		)
+		(instances
+			(project "smart_soldering_iron"
+				(path "/2df86fbf-058b-45fc-8204-866599907949/63b7c06e-9066-41e6-8478-c4bea396f7f1"
+					(reference "R?")
+					(unit 1)
+				)

Commit message: COMPLETED CIRCUIT DIAGRAM
Parts:
- added C25: 10u, Capacitor_SMD:C_0603_1608Metric, symbol Device:C
- added C27: 100u 35V, Capacitor_SMD:C_1206_3216Metric, symbol Device:C
- added C28: 10u 35V, Capacitor_SMD:C_0603_1608Metric, symbol Device:C
- added C35: 100n, Capacitor_SMD:C_0603_1608Metric, symbol Device:C
- added D11: D_Zener, symbol Device:D_Zener
- added D12, D13: D_SchottKy, symbol Device:D_Schottky
- added D7: D, symbol Device:D
- added J3: Conn_01x02_Pin, symbol Connector:Conn_01x02_Pin
- added Q10: ~, smart_soldering_iron:AON7410_POWER_N_MOS_DFN-8_L3.0-W3.0-P0.65-BL, symbol smart_soldering_iron:AON7410
- added Q11: ~, smart_soldering_iron:S8050_TRANSIS_25V_0.5A_npn_SOT-23-3_L2.9-W1.3-P1.90-LS2.4-BR, symbol smart_soldering_iron:S8050
- added R43: 1K, Resistor_SMD:R_0805_2012Metric, symbol Device:R
- added R44: 10K, Resistor_SMD:R_0603_1608Metric, symbol Device:R
- added R50: 56K, Resistor_SMD:R_0603_1608Metric, symbol Device:R
- added R51: 1K, Resistor_SMD:R_0603_1608Metric, symbol Device:R
- added R52: 75K, Resistor_SMD:R_0603_1608Metric, symbol Device:R
- added R53: 0.01, symbol Device:R
- added U9: ~, smart_soldering_iron:LM321_SOT-23-5_L3.0-W1.7-P0.95-LS2.8-BR, symbol smart_soldering_iron:LM321_C5252901
- C12, C13, C14, C15, C16, C17, C18, C19, C22: renamed from C?; footprint (none) -> Capacitor_SMD:C_0603_1608Metric
- C20, C21: renamed from C?; footprint (none) -> Capacitor_SMD:C_0805_2012Metric
- L1: renamed from L?; value 6.8u -> 4.7u
- R13: renamed from R?; value 10k -> 10K; footprint (none) -> Resistor_SMD:R_0603_1608Metric
- R14, R15: renamed from R?; value 1k -> 1K; footprint (none) -> Resistor_SMD:R_0603_1608Metric
- R16: renamed from R?; value 1k -> 10K; footprint (none) -> Resistor_SMD:R_0603_1608Metric
- R17: renamed from R?; footprint (none) -> Resistor_SMD:R_0603_1608Metric
- R18: renamed from R?; value 10k -> 9K; footprint (none) -> Resistor_SMD:R_0603_1608Metric
- R19: renamed from R?; value 10k -> 30K; footprint (none) -> Resistor_SMD:R_0603_1608Metric
- U4: renamed from U?; footprint CH340C:SO016 -> smart_soldering_iron:CH340C_SO016
- U6: renamed from U?; footprint ProLib_pcs_2025-10-04:TSOT-23-6_L2.9-W1.6-P0.95-LS2.8-BR -> smart_soldering_iron:DIODES AP63300WU-7_buck_TSOT-23-6_L2.9-W1.6-P0.95-LS2.8-BR
- U7: renamed from U?; footprint ProLib_pcs_2025-10-04:SOT-23-3_L3.0-W1.7-P0.95-LS2.9-BR -> smart_soldering_iron:XC6206P332MR_SOT-23-3_L2.9-W1.3-P1.90-LS2.4-BR
- USB1: renamed from USB?; footprint ProLib_pcs_2025-10-03:USB-C-SMD_TYPE-C-6PIN-2MD-073 -> smart_soldering_iron:USB-C-SMD_TYPE-C-6PIN-2MD-073
- gave numbers to parts that had none: 2
Connections:
- net GND: now also C27.2, C28.2, C35.2, Q11.2 (E), R51.1, R53.2, U9.2 (V-)
- net Vin: now also C27.1, C28.1, D13.2 (A); no longer C16.1, U6.2 (EN), U6.3 (VIN)
- net at U5.4 (DP): now also U5.5 (DM)
- net D0_rxd renamed D0_RXD
- net D1_txd renamed D1_TXD
- net cfg1 renamed CFG1
- net cfg2 renamed CFG2
- net cfg3 renamed CFG3
- net pg renamed PG
- net vcc_3v3 renamed VCC_3V3
- net vcc_5v renamed VCC_5V
- net VCC_5V: now also U9.5 (V+)
- new net: C25.2, D7.1 (K), R43.1
- new net: D12.1 (K), D13.1 (K), D7.2 (A), Q10.5 (D), Q10.6 (D), Q10.7 (D), Q10.8 (D), Q10.9 (D)
- new net: C35.1, R50.2, U9.1 (IN+)
- new net: Q11.1 (B), R44.2
- new net: D11.1 (K), Q10.4 (G), Q11.3 (C), R43.2
- new net: R51.2, R52.1, U9.3 (IN-)
- new net 2S: D12.2 (A)
- new net 2S_MOS_OUT: C16.1, U6.2 (EN), U6.3 (VIN)
- new net TIP+: C25.1, D11.2 (A), J3.2 (Pin_2), Q10.1 (S), Q10.2 (S), Q10.3 (S)
- new net TIP-: J3.1 (Pin_1), R50.1, R53.1
- new net TIP_AMP_SENSE: R52.2, U9.4 (OUT)
- new net TIP_MOS: R44.1
- no-connect marks 12 -> 10
Other:
- note removed: "component values not confirmed"
- moved on the sheet: C12, C13, C14, C15, D3, R13, R14, R15, R16, R17, U4, U5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
